File: KiCad/MiProyecto.sch (KiCad schematic (older format))
At the start: 30 parts, among them SW1 SW_DIP_x01, SW1 SW_Push, SW2 SW_Push, U1 7805, U2 STM32F407VGT, U3 Display7SEG, U3 HC-05

Commit message: Add files via upload
Parts:
- R1: value 200 -> 220
Connections:
- net at C2.1, DS1.15 (LED+), DS1.2 (VDD)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: now also POT1.1
- net at R1.1: now also U3.~; no longer U2.~
- net at R1.2: now also U2.~; no longer U3.~
- net at U2.~: now also SW2.1; no longer POT1.1
- net at U3.~: no longer U2.~
- new net: U2.~, U3.~ (x8)
- now unconnected: U3.~
Other:
- moved on the sheet: POT1, R1, U3
